File: serdes-rf-hdmi.kicad_pcb (KiCad board)
At the start: 4 copper layers, 53.5 x 25 mm, 27 parts, among them J1 HDMI_A, J2 SMA, J3 SMA

Commit message: Fix bandpass filter and add coupling caps.  Update image and README.
Parts:
- added C10: 0.1uF, Capacitor_SMD:C_0603_1608Metric, F.Cu at (138.2, 78.8)
- added C11: 0.1uF, Capacitor_SMD:C_0603_1608Metric, F.Cu at (138.2, 87.2)
- added REF**: OSHW-Logo2_7.3x6mm_SilkScreen, Symbol:OSHW-Logo2_7.3x6mm_SilkScreen, B.Cu at (163.0, 84.5)
- moved C2 4.50 mm to (142.8, 79.8)
- moved C3 4.50 mm to (142.8, 88.2)
- moved C4 4.50 mm to (146.8, 79.8), turned to 270 degrees
- moved C5 4.50 mm to (146.8, 88.2), turned to 270 degrees
- moved C6 4.50 mm to (150.8, 79.8)
- moved C7 4.50 mm to (150.8, 88.2)
- moved C8 4.50 mm to (154.8, 79.8), turned to 270 degrees
- moved C9 4.50 mm to (154.8, 88.2), turned to 270 degrees
- moved G1 1.58 mm to (160.0, 84.5)
- moved L1 0.50 mm to (140.8, 79.8)
- moved L2 0.50 mm to (140.8, 88.2)
- moved L3 0.50 mm to (144.8, 79.8), turned to 270 degrees
- moved L4 0.50 mm to (144.8, 88.2), turned to 270 degrees
- moved L5 0.50 mm to (148.8, 79.8)
- moved L6 0.50 mm to (148.8, 88.2)
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Connections:
- C2 pad 1: Net-(C2-Pad1) -> Net-(C10-Pad2)
- C3 pad 1: Net-(C3-Pad1) -> Net-(C11-Pad2)
- C4 pad 2: Net-(C2-Pad1) -> Net-(C4-Pad2)
- C5 pad 2: Net-(C3-Pad1) -> Net-(C5-Pad2)
- C6 pad 1: Net-(C6-Pad1) -> Net-(C4-Pad1)
- C7 pad 1: Net-(C7-Pad1) -> Net-(C5-Pad1)
- C8 pad 1: Net-(C8-Pad1) -> /rfa
- C8 pad 2: Net-(C6-Pad1) -> Net-(C8-Pad2)
- C9 pad 1: Net-(C9-Pad1) -> /rfb
- C9 pad 2: Net-(C7-Pad1) -> Net-(C9-Pad2)
- J2 pad 1: Net-(J2-Pad1) -> /rfb
- J3 pad 1: Net-(J3-Pad1) -> /rfa
- L1 pad 1: Net-(C2-Pad1) -> Net-(C10-Pad2)
- L2 pad 1: Net-(C3-Pad1) -> Net-(C11-Pad2)
- L3 pad 1: Net-(C4-Pad1) -> Net-(C10-Pad2)
- L3 pad 2: Net-(C6-Pad1) -> Net-(C4-Pad2)
- L4 pad 1: Net-(C5-Pad1) -> Net-(C11-Pad2)
- L4 pad 2: Net-(C7-Pad1) -> Net-(C5-Pad2)
- L5 pad 1: Net-(C6-Pad1) -> Net-(C4-Pad1)
- L6 pad 1: Net-(C7-Pad1) -> Net-(C5-Pad1)
- L7 pad 1: Net-(C8-Pad1) -> Net-(C4-Pad1)
- L7 pad 2: Net-(J3-Pad1) -> Net-(C8-Pad2)
- L8 pad 1: Net-(C9-Pad1) -> Net-(C5-Pad1)
- L8 pad 2: Net-(J2-Pad1) -> Net-(C9-Pad2)
- TR1 pad 4: Net-(C2-Pad1) -> Net-(C10-Pad1)
- TR2 pad 4: Net-(C3-Pad1) -> Net-(C11-Pad1)
Routing:
- net Net-(J2-Pad1): track 19.5 -> 0.00 mm
- net Net-(J3-Pad1): track 18.1 -> 0.00 mm
- net /rfb: track 0.00 -> 17.0 mm
- net /rfa: track 0.00 -> 15.5 mm
- net Net-(C2-Pad1): track 7.21 -> 0.00 mm
- net Net-(C3-Pad1): track 6.99 -> 0.00 mm
- net Net-(C10-Pad2): track 0.00 -> 6.24 mm
- net Net-(C7-Pad1): track 6.02 -> 0.00 mm
- net Net-(C11-Pad2): track 0.00 -> 6.02 mm
- net Net-(C6-Pad1): track 6.01 -> 0.00 mm
- net /rfb-: track 15.6 -> 19.9 mm
- net Net-(C5-Pad1): track 2.01 -> 6.02 mm
- net Net-(C4-Pad1): track 2.01 -> 6.01 mm
- net Net-(C11-Pad1): track 0.00 -> 2.14 mm
- net Net-(C10-Pad1): track 0.00 -> 2.14 mm
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Other:
- net class 50ohm added: clearance 0.62, trace_width 0.31, via_dia 0.8, via_drill 0.4
- net class Power added: clearance 0.5, trace_width 0.5, via_dia 0.8, via_drill 0.4
- board text added: "®©®"

Commit message: Trivial changes to layout.
Parts:
- moved REF** 2.30 mm to (160.8, 84.0)
Routing:
- net GND: track 19.6 -> 16.4 mm, vias 52 -> 51
